File: Snacks65/Snacks65.kicad_pcb (KiCad board)
At the start: 2 copper layers, 147 parts, among them J1 Conn_02x03_Odd_Even, J2 Conn_01x04_Female, SW1 SW_PUSH, SW10 1U, SW11 1.25U, SW12 1U, SW13 1U, SW14 1U, SW15 1U, SW16 1.25U, SW17 1U, SW18 1U, SW19 1U, SW2 1U, SW20 1U, SW21 1U, SW22 1U, SW23 1U, SW24 1U, SW25 1U, SW26 1U, SW27 1U, SW28 1U, SW29 1U, SW3 1.5U, SW30 1U, SW31 1U, SW32 1U, SW33 6.25U, SW34 1U, SW35 1U, SW36 1U, SW37 1U, SW38 1U, SW39 1U, SW4 1.75U, SW40 1U, SW41 1U, SW42 1U, SW43 1U, SW44 1U, SW45 1U, SW46 1U, SW47 1U, SW48 1U, SW49 1U, SW5 1.25U, SW51 1U, SW52 1U, SW53 1U, SW54 1U, SW55 1.25U, SW56 1U, SW57 1U, SW58 2.25, SW59 1.75U, SW6 1.25U, SW60 1.25U, SW61 1U, SW62 1.5U, SW63 1U, SW64 1.25U, SW65 1U, SW66 2.25, SW67 2.75U, SW68 2U, SW69 1U, SW7 1U, SW70 1U, SW71 1U, SW72 1U, SW73 1U, SW74 1U, SW75 1U, SW76 1U, SW8 1U, SW9 1U, U1 ATmega32U4-AU, Y1 Resonator_Small, Y2 Crystal_GND24

Commit message: 7/24
Parts:
- removed C1, C10, C8: 1uF, Capacitor_SMD:C_0805_2012Metric
- removed C11, C12, C2, C3, C5, C9: 100nF, Capacitor_SMD:C_0805_2012Metric
- removed C13, C6: 4.7uF, Capacitor_SMD:C_0805_2012Metric
- removed C14: 10uF, Capacitor_SMD:C_0805_2012Metric
- removed C4, C7: 18pF, Capacitor_SMD:C_0805_2012Metric
- removed D29: LED, LED_THT:LED_D3.0mm
- removed D39, D40: BAV70, Package_TO_SOT_SMD:SOT-23
- removed F1: ASMD1206-200, Fuse:Fuse_1206_3216Metric
- removed J2: Conn_01x04_Female, random-keyboard-parts:JST-SR-4
- removed R10: 12kΩ, Resistor_SMD:R_0805_2012Metric
- removed R11: 2.2k, Resistor_SMD:R_0805_2012Metric
- removed R3, R4: 10kΩ, Resistor_SMD:R_0805_2012Metric
- removed R5: 330Ω, Resistor_SMD:R_0805_2012Metric
- removed R6, R7: 5.1kΩ, Resistor_SMD:R_0805_2012Metric
- removed R8: 100kΩ, Resistor_SMD:R_0805_2012Metric
- removed R9: 100k, Resistor_SMD:R_0805_2012Metric
- removed SW73, SW76: 1U, MX_Alps_Hybrid:MX-1U-NoLED
- removed U1: ATmega32U4-AU, Package_QFP:TQFP-44_10x10mm_P0.8mm
- removed USB1: HRO-TYPE-C-31-M-12, Type-C:HRO-TYPE-C-31-M-12-HandSoldering
- removed Y1: Resonator_Small, proj_local:Resonator_SMD_muRata_CSTxExxV-3Pin_3.0x1.1mm_HandSoldering_Compact
- removed Y2: Crystal_GND24, keyboard_parts:FA-238
- added A1: Adafruit_Feather_32u4_BluefruitLE, feather:Adafruit_Feather, F.Cu at (445.3, 31.0)
- D1, D10, D11, D12, D13, D14, D15, D16, D17, D18, D19, D2, D20, D21, D22, D23, D24, D25, D26, D27, D28, D3, D30, D31, D32, D33, D34, D35, D36, D37, D38, D4, D5, D6, D7, D8, D9: moved to B.Cu
- J1: value Conn_02x03_Odd_Even -> Sensor Connector; footprint Connector_PinHeader_2.54mm:PinHeader_2x03_P2.54mm_Vertical -> Connector_FFC-FPC:Hirose_FH12-6S-0.5SH_1x06-1MP_P0.50mm_Horizontal
- R1, R2: value 22Ω -> 4.7k
- SW1: value SW_PUSH -> SW_SPDT; footprint random-keyboard-parts:SKQG-1155865 -> Custom_Footprints:Slide_Switch_SPDT_ThroughHole
- moved D1 607.1 mm to (38.1, 27.8), turned to 270 degrees
- moved D2 596.6 mm to (45.2, 46.8), turned to 270 degrees
- moved D5 586.2 mm to (42.9, 104.0), turned to 270 degrees
- moved D3 585.4 mm to (49.2, 65.9), turned to 270 degrees
- moved D6 572.2 mm to (76.2, 27.8), turned to 270 degrees
- moved D8 544.1 mm to (90.5, 65.9), turned to 270 degrees
- moved D4 541.3 mm to (61.9, 84.9), turned to 270 degrees
- moved D9 535.7 mm to (81.0, 84.9), turned to 270 degrees
- moved D7 519.1 mm to (85.7, 46.8), turned to 270 degrees
- moved D10 518.2 mm to (90.6, 103.8), turned to 270 degrees
- moved D13 513.2 mm to (128.6, 65.9), turned to 270 degrees
- moved D11 507.8 mm to (114.3, 27.8), turned to 270 degrees
- moved D12 495.4 mm to (123.8, 46.8), turned to 270 degrees
- moved D14 482.3 mm to (119.1, 84.7), turned to 270 degrees
- moved D15 463.9 mm to (152.4, 27.8), turned to 270 degrees
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Connections:
- D24 pad 3: Net-(D24-Pad3) -> COL5
- D25 pad 3: Net-(D24-Pad3) -> COL5
- D26 pad 3: Net-(D24-Pad3) -> COL5
- D27 pad 3: Net-(D24-Pad3) -> COL5
- D28 pad 3: Net-(D24-Pad3) -> COL5
- J1 pad 1: ROW3 -> SDA
- J1 pad 2: +5V -> SCL
- J1 pad 3: ROW1 -> +3V3
- J1 pad 4: ROW2 -> GND
- J1 pad 6: GND -> RDY
- R1 pad 1: Net-(R1-Pad1) -> +3V3
- R1 pad 2: DOWN1_D- -> SDA
- R2 pad 1: Net-(R2-Pad1) -> +3V3
- R2 pad 2: DOWN1_D+ -> SCL
- SW1 pad 2: Net-(J1-Pad5) -> /EN
- SW1 pad 3: (no net) -> Net-(SW1-Pad3)
- SW55 pad 1: Net-(D28-Pad2) -> Net-(D28-Pad1)
- SW55 pad 2: ROW9 -> ROW8
- SW58 pad 1: Net-(D32-Pad1) -> Net-(D32-Pad2)
- SW60 pad 1: Net-(D34-Pad1) -> Net-(D28-Pad2)
- SW60 pad 2: ROW8 -> ROW9
- SW64 pad 1: Net-(D34-Pad2) -> Net-(D34-Pad1)
- SW64 pad 2: ROW9 -> ROW8
- SW69 pad 1: Net-(D37-Pad1) -> Net-(D37-Pad2)
- SW70 pad 1: Net-(D38-Pad1) -> Net-(D34-Pad2)
- SW70 pad 2: ROW8 -> ROW9
- SW71 pad 1: Net-(D36-Pad1) -> Net-(D36-Pad2)
- SW74 pad 1: Net-(D38-Pad2) -> Net-(D38-Pad1)
- SW74 pad 2: ROW9 -> ROW8
- SW75 pad 1: Net-(D40-Pad1) -> Net-(D38-Pad2)
- SW75 pad 2: ROW8 -> ROW9
Routing:
- net COL1: track 0.00 -> 448.3 mm, vias 0 -> 1
- net COL0: track 0.00 -> 442.0 mm, vias 0 -> 2
- net ROW6: track 0.00 -> 425.1 mm
- net ROW8: track 0.00 -> 420.9 mm
- net ROW7: track 0.00 -> 410.7 mm
- net ROW9: track 0.00 -> 407.7 mm
- net ROW0: track 0.00 -> 404.9 mm
- net ROW1: track 0.00 -> 398.5 mm
- net ROW4: track 0.00 -> 396.3 mm
- net ROW2: track 0.00 -> 394.7 mm
- net ROW3: track 0.00 -> 386.1 mm
- net COL2: track 0.00 -> 382.7 mm, vias 0 -> 1
- net ROW5: track 0.00 -> 377.7 mm
- net COL3: track 0.00 -> 365.2 mm, vias 0 -> 1
- net COL4: track 0.00 -> 302.4 mm, vias 0 -> 1
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Other:
- board outline added: 435 x 100 mm
- net class PWR added: clearance 0.2, trace_width 0.381, via_dia 0.8, via_drill 0.4

Commit message: 7-27
Parts:
- removed D35, D36, D37, D38: BAV70, Package_TO_SOT_SMD:SOT-23
- removed SW61, SW65, SW69, SW70, SW71, SW72, SW74, SW75: 1U, MX_Alps_Hybrid:MX-1U-NoLED
- A1, J1, R1, R2, SW1: moved to B.Cu
- moved A1 111.3 mm to (334.2, 24.6), turned to 180 degrees
- moved R2 108.9 mm to (340.7, 51.1), turned to 180 degrees
- moved J1 107.0 mm to (344.5, 42.1)
- moved R1 104.0 mm to (340.7, 53.8), turned to 180 degrees
- moved SW1 36.5 mm to (346.9, 19.8)
Connections:
- A1 pad 10: COL5 -> COL3
- A1 pad 11: COL6 -> COL1
- A1 pad 12: COL7 -> ROW4
- A1 pad 13: ROW3 -> ROW6
- A1 pad 14: ROW2 -> ROW8
- A1 pad 15: ROW1 -> ROW9
- A1 pad 19: COL0 -> ROW7
- A1 pad 20: ROW4 -> ROW5
- A1 pad 21: ROW5 -> COL0
- A1 pad 22: ROW6 -> COL2
- A1 pad 23: ROW7 -> COL4
- A1 pad 24: ROW8 -> COL6
- A1 pad 25: ROW9 -> ROW2
- A1 pad 6: COL1 -> ROW0
- A1 pad 7: COL2 -> ROW1
- A1 pad 8: COL3 -> ROW3
- A1 pad 9: COL4 -> COL5
Routing:
- net COL7: track 209.3 -> 0.00 mm, vias 1 -> 0
- net COL2: track 382.7 -> 258.6 mm
- net COL4: track 302.4 -> 184.4 mm
- net COL6: track 258.9 -> 147.0 mm
- net ROW7: track 410.7 -> 303.7 mm
- net COL1: track 448.3 -> 342.0 mm
- net ROW5: track 377.7 -> 272.7 mm
- net ROW2: track 394.7 -> 290.5 mm
- net COL3: track 365.2 -> 265.0 mm
- net COL5: track 281.5 -> 187.4 mm
- net ROW6: track 425.1 -> 332.3 mm
- net ROW3: track 386.1 -> 298.0 mm
- net ROW9: track 407.7 -> 321.2 mm
- net ROW1: track 398.5 -> 315.5 mm
- net ROW4: track 396.3 -> 314.3 mm
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- added copper zone on B.Cu, net (none)
- added copper zone on F.Cu, net (none)
- added copper zone on B.Cu, net GND
- added copper zone on F.Cu, net GND
Other:
- board size 435 x 100 mm -> 336.6 x 100 mm

Commit message: 8/29
Parts:
- added D29: BAV70, Package_TO_SOT_SMD:SOT-23, B.Cu at (309.6, 27.8)
- added D35: BAV70, Package_TO_SOT_SMD:SOT-23, B.Cu at (309.6, 46.8)
- added D36: BAV70, Package_TO_SOT_SMD:SOT-23, B.Cu at (309.6, 85.1)
- added D37: BAV70, Package_TO_SOT_SMD:SOT-23, B.Cu at (333.4, 103.2)
- added SW50: 1U, MX_Alps_Hybrid:MX-1U-NoLED, F.Cu at (304.8, 105.6)
- added SW61: 1U, MX_Alps_Hybrid:MX-1U-NoLED, F.Cu at (323.9, 29.4)
- added SW65: 1U, MX_Alps_Hybrid:MX-1U-NoLED, F.Cu at (323.9, 48.4)
- added SW69: 1U, MX_Alps_Hybrid:MX-1U-NoLED, F.Cu at (323.9, 86.5)
- added SW70: 1U, MX_Alps_Hybrid:MX-1U-NoLED, F.Cu at (323.9, 105.6)
- added SW71: 1U, MX_Alps_Hybrid:MX-1U-NoLED, F.Cu at (342.9, 105.6)
- added U1: MCP23017_SP, Package_DIP:DIP-28_W7.62mm, F.Cu at (339.7, 57.1)
- moved A1 113.0 mm to (445.3, 45.2), turned to 90 degrees
- moved J1 33.2 mm to (323.1, 67.5)
Connections:
- A1 pad 11: COL1 -> Net-(A1-Pad11)
- A1 pad 12: ROW4 -> Net-(A1-Pad12)
- A1 pad 13: ROW6 -> Net-(A1-Pad13)
- A1 pad 14: ROW8 -> COL2
- A1 pad 15: ROW9 -> INTB
- A1 pad 22: COL2 -> ROW8
- A1 pad 23: COL4 -> COL5
- A1 pad 24: COL6 -> ROW3
- A1 pad 8: ROW3 -> COL6
- A1 pad 9: COL5 -> COL4
Routing:
- net COL7: track 0.00 -> 134.4 mm
- net COL5: track 187.4 -> 86.1 mm, vias 1 -> 0
- net ROW1: track 315.5 -> 369.9 mm
- net SCL: track 52.9 -> 0.00 mm
- net SDA: track 52.6 -> 0.00 mm
- net ROW2: track 290.5 -> 244.4 mm
- net +3V3: track 44.4 -> 0.00 mm
- net ROW3: track 298.0 -> 256.6 mm
- net /EN: track 41.1 -> 0.00 mm
- net GND: track 38.9 -> 0.14 mm
- net COL1: track 342.0 -> 308.5 mm
- net ROW6: track 332.3 -> 304.4 mm
- net ROW4: track 314.3 -> 286.4 mm
- net ROW9: track 321.2 -> 293.7 mm
- net ROW8: track 341.2 -> 314.6 mm
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- removed copper zone on B.Cu, net (none)
- removed copper zone on F.Cu, net (none)
- removed copper zone on B.Cu, net GND
- removed copper zone on F.Cu, net GND
Other:
- board size 336.6 x 100 mm -> 435.2 x 100 mm
